Commit message: progress towards DaVinci gazebo model; see gazebo_notes_9_12 for start-up need to modify traj_streamer to talk to davinci joints

File: dvrk_model/model/wsntest_psm_debug.base.urdf (robot description, URDF)
Before this commit: robot dvrk_psm, 0 links, 0 joints
Links:
- added link outer_insertion_link, mass 0.1; visual mesh filename=package://dvrk_model/meshes/psm/outer_insertion.dae
- added link outer_pitch_back_link, mass 0.1; visual mesh filename=package://dvrk_model/meshes/psm/outer_pitch_back.dae
- added link outer_pitch_bottom_link, mass 0.1; visual mesh filename=package://dvrk_model/meshes/psm/outer_pitch_bottom.dae
- added link outer_pitch_front_link, mass 0.1; visual mesh filename=package://dvrk_model/meshes/psm/outer_pitch_front.dae
- added link outer_pitch_link, mass 0.1
- added link outer_pitch_top_link, mass 0.1; visual mesh filename=package://dvrk_model/meshes/psm/outer_pitch_top.dae
- added link outer_yaw_link, mass 0.1; visual mesh filename=package://dvrk_model/meshes/psm/outer_yaw.dae
- added link psm_base_link, mass 1; visual mesh filename=package://dvrk_model/meshes/psm/psm_base.dae
- added link tool_main_link, mass 0.1; visual mesh filename=package://dvrk_model/meshes/psm/tool_main.dae
- added link tool_wrist_link, mass 0.1; visual mesh filename=package://dvrk_model/meshes/psm/tool_wrist_link.dae
- added link tool_wrist_shaft_link, mass 0.1; visual mesh filename=package://dvrk_model/meshes/psm/tool_wrist_shaft_link.dae
- added link world
Joints:
- added joint glue_robot_to_world: type fixed, parent world, child psm_base_link, origin xyz=0 0 0.5 rpy=0 0 0
- added joint outer_insertion_joint: type prismatic, parent outer_pitch_link, child tool_main_link, origin xyz=0 0.4318 0 rpy=1.5708 0 0, axis 0 0 1, limit lower=-0.3 upper=0.3 effort=1000 velocity=.4
- added joint outer_pitch_joint: type revolute, parent outer_yaw_link, child outer_pitch_link, origin xyz=0 0 0 rpy=-1.5708 -1.5708 0, axis 0 0 1, limit lower=-0.7854 upper=0.7854 effort=1000 velocity=.4
- added joint outer_pitch_joint_1: type continuous, parent outer_yaw_link, child outer_pitch_back_link, origin xyz=0 0.0295 0.5185 rpy=-1.5708 -1.5708 0, axis 0 0 1, limit lower=-0.7854 upper=0.7854 effort=1000 velocity=.4
- added joint outer_pitch_joint_2: type continuous, parent outer_yaw_link, child outer_pitch_front_link, origin xyz=0 0.0295 0.4285 rpy=-1.5708 -1.5708 0, axis 0 0 1, limit lower=-0.7854 upper=0.7854 effort=1000 velocity=.4, mimic joint=outer_pitch_joint multiplier=1
- added joint outer_pitch_joint_3: type continuous, parent outer_pitch_back_link, child outer_pitch_bottom_link, origin xyz=0.04178 0.15007 -0.0137 rpy=0 0 0, axis 0 0 1, limit lower=-0.7854 upper=0.7854 effort=1000 velocity=.4, mimic joint=outer_pitch_joint multiplier=-1
- added joint outer_pitch_joint_4: type continuous, parent outer_pitch_back_link, child outer_pitch_top_link, origin xyz=0.04209 0.18695 -0.02412 rpy=0 0 0, axis 0 0 1, limit lower=-0.7854 upper=0.7854 effort=1000 velocity=.4, mimic joint=outer_pitch_joint multiplier=-1
- added joint outer_pitch_joint_5: type continuous, parent outer_pitch_bottom_link, child outer_insertion_link, origin xyz=-0.520 0 -0.0155 rpy=0 0 0, axis 0 0 1, limit lower=-0.7854 upper=0.7854 effort=1000 velocity=.4, mimic joint=outer_pitch_joint multiplier=1
- added joint outer_roll_joint: type revolute, parent tool_main_link, child tool_wrist_link, origin xyz=0 0 0.4162 rpy=0 0 0, axis 0 0 1, limit lower=-2.2689 upper=2.2689 effort=1000 velocity=.4
- added joint outer_roll_shaft_joint: type fixed, parent tool_wrist_link, child tool_wrist_shaft_link, origin xyz=0 0 0.0 rpy=0 0 0, axis 0 0 1
- added joint outer_yaw_joint: type revolute, parent psm_base_link, child outer_yaw_link, origin xyz=0.0 0.0 0.0 rpy=0 -1.5708 1.5708, axis 0 0 1, limit lower=-1.5707 upper=1.5707 effort=1000 velocity=.4
