Commit message: hand off peg program...shifted psm's

File: dvrk_model/model/wsn_both_psms.urdf.xacro (robot description, xacro)
@@ -17,5 +17,5 @@
       <parent link="camera"/>
       <child link="right_camera_link"/>
-      <origin rpy="0.0 1.5708 1.5708" xyz="-0.006 0.0 0.5"/>
+      <origin rpy="0.0 1.5708 1.5708" xyz="-0.005 0.0 0.5"/>
   </joint>
   <link name="right_camera_link">
@@ -37,5 +37,5 @@
       <parent link="camera"/>
       <child link="left_camera_link"/>
-      <origin rpy="0.0 1.5708 1.5708" xyz="0.006 0.00 0.5"/>
+      <origin rpy="0.0 1.5708 1.5708" xyz="0.005 0.00 0.5"/>
   </joint>
   <link name="left_camera_link">
@@ -57,9 +57,9 @@
       prefix="one_"
       parent_link="camera"
-      xyz="-0.15 0.0 0.5" rpy="0.0 0.0 3.1415926"/>
+      xyz="-0.15 0.05 0.5" rpy="0.0 0.0 3.1415926"/>
   <xacro:psm_sca
       prefix="two_"
       parent_link="camera"
-      xyz="0.15 0.0 0.5" rpy="0.0 0.0 3.1415926"/>
+      xyz="0.15 0.05 0.5" rpy="0.0 0.0 3.1415926"/>
   <!-- ros_control plugin -->
   <gazebo>
