Commit message: added checkerboard for calib in simu added red spheres at tips of grippers

File: dvrk_model/model/gazebo_psm.tool.sca.urdf.xacro (robot description, xacro)
@@ -3,4 +3,6 @@
   <!-- This file contains different tool urdf -->
   <xacro:include filename="$(find dvrk_model)/model/common.urdf.xacro"/>
+  <xacro:property name="GazeboRed"       value="1 0 0 1"/>
+  <material name="GazeboRed">      <color rgba="${GazeboRed}"/></material>
   <!-- sca  -->
   <xacro:macro name="psm_tool_sca" params="prefix">
@@ -142,5 +144,16 @@
       <origin rpy="0 ${PI/2} ${PI/2}" xyz="0 0.0102 0"/>
     </joint>
-    <link name="${prefix}tool_tip_link"/>
+    <link name="${prefix}tool_tip_link">
+     <visual>
+      <geometry>
+          <!-- put a fiducial, a sphere, at the tool tips -->
+        <sphere radius="0.001"/>
+      </geometry>
+    </visual>
+    </link>
+ <!--this colors the tool-tip fiducial red; oddly, this shows up in the camera view, but NOT in the rviz view -->
+  <gazebo reference="${prefix}tool_tip_link">
+    <material>Gazebo/Red</material>
+  </gazebo>
  <transmission name="${prefix}tran5">
     <type>transmission_interface/SimpleTransmission</type>

File: dvrk_model/model/wsn_both_psms.urdf.xacro (robot description, xacro)
@@ -9,8 +9,48 @@
       <parent link="world"/>
       <child link="camera"/>
-      <origin rpy="0.0 0.0 0.0" xyz="0.0 0.0 0.0"/>
+      <origin rpy="0.0 0.0 0.0" xyz="0.0 0.0 0.5"/>
   </joint>
-  <link name="camera">
-  <origin rpy="0.0 0.0 0.0" xyz="0.0 0.2 0.8"/>
+    <link name="camera">
+    <origin rpy="0.0 0.0 0.0" xyz="0.0 0.0 0.8"/>
+  </link>
+  <joint name="camera_joint" type="fixed">
+      <parent link="camera"/>
+      <child link="right_camera_link"/>
+      <origin rpy="0.0 1.5708 1.5708" xyz="-0.006 0.0 0.5"/>
+  </joint>
+  <link name="right_camera_link">
+    <visual>
+      <origin xyz="0 0 0.0" rpy="0 0 0"/>
+      <geometry>
+        <box size="0.03 0.01 0.01"/>
+      </geometry>
+      <material name="red"/>
+    </visual>
+    <inertial>
+      <mass value="1e-5" />
+      <origin xyz="0 0 0" rpy="0 0 0"/>
+      <inertia ixx="1e-6" ixy="0" ixz="0" iyy="1e-6" iyz="0" izz="1e-6" />
+    </inertial>
+  <!--origin rpy="0.0 0.0 0.0" xyz="0.0 0.2 0.8"/-->
+  </link>
+    <joint name="left_camera_joint" type="fixed">
+      <parent link="camera"/>
+      <child link="left_camera_link"/>
+      <origin rpy="0.0 1.5708 1.5708" xyz="0.006 0.00 0.5"/>
+  </joint>
+  <link name="left_camera_link">
+    <visual>
+      <origin xyz="0 0 0.0" rpy="0 0 0"/>
+      <geometry>
+        <box size="0.03 0.01 0.01"/>
+      </geometry>
+      <material name="red"/>
+    </visual>
+    <inertial>
+      <mass value="1e-5" />
+      <origin xyz="0 0 0" rpy="0 0 0"/>
+      <inertia ixx="1e-6" ixy="0" ixz="0" iyy="1e-6" iyz="0" izz="1e-6" />
+    </inertial>
+  <!--origin rpy="0.0 0.0 0.0" xyz="0.0 0.2 0.8"/-->
   </link>
   <xacro:psm_sca
@@ -29,3 +69,83 @@
     </plugin>
   </gazebo>
+  <!-- camera -->
+  <gazebo reference="right_camera_link">
+    <sensor type="camera" name="right_camera">
+      <update_rate>30.0</update_rate>
+      <camera name="right_camera">
+        <horizontal_fov>0.6</horizontal_fov>
+        <image>
+          <width>640</width>
+          <height>480</height>
+          <format>R8G8B8</format>
+        </image>
+        <clip>
+          <near>0.005</near>
+          <far>0.9</far>
+        </clip>
+        <noise>
+          <type>gaussian</type>
+          <!-- Noise is sampled independently per pixel on each frame.
+               That pixel's noise value is added to each of its color
+               channels, which at that point lie in the range [0,1]. -->
+          <mean>0.0</mean>
+          <stddev>0.007</stddev>
+        </noise>
+      </camera>
+      <plugin name="camera_controller" filename="libgazebo_ros_camera.so">
+        <alwaysOn>true</alwaysOn>
+        <updateRate>0.0</updateRate>
+        <cameraName>davinci/right_camera</cameraName>
+        <imageTopicName>image_raw</imageTopicName>
+        <cameraInfoTopicName>camera_info</cameraInfoTopicName>
+        <frameName>right_camera_link</frameName>
+        <hackBaseline>0.07</hackBaseline>
+        <distortionK1>0.0</distortionK1>
+        <distortionK2>0.0</distortionK2>
+        <distortionK3>0.0</distortionK3>
+        <distortionT1>0.0</distortionT1>
+        <distortionT2>0.0</distortionT2>
+      </plugin>
+    </sensor>
+  </gazebo>
+   <!-- left camera -->
+  <gazebo reference="left_camera_link">
+    <sensor type="camera" name="left_camera">
+      <update_rate>30.0</update_rate>
+      <camera name="left_camera">
+        <horizontal_fov>0.6</horizontal_fov>
+        <image>
+          <width>640</width>
+          <height>480</height>
+          <format>R8G8B8</format>
+        </image>
+        <clip>
+          <near>0.005</near>
+          <far>0.9</far>
+        </clip>
+        <noise>
+          <type>gaussian</type>
+          <!-- Noise is sampled independently per pixel on each frame.
+               That pixel's noise value is added to each of its color
+               channels, which at that point lie in the range [0,1]. -->
+          <mean>0.0</mean>
+          <stddev>0.007</stddev>
+        </noise>
+      </camera>
+      <plugin name="camera_controller" filename="libgazebo_ros_camera.so">
+        <alwaysOn>true</alwaysOn>
+        <updateRate>0.0</updateRate>
+        <cameraName>davinci/left_camera</cameraName>
+        <imageTopicName>image_raw</imageTopicName>
+        <cameraInfoTopicName>camera_info</cameraInfoTopicName>
+        <frameName>left_camera_link</frameName>
+        <hackBaseline>0.07</hackBaseline>
+        <distortionK1>0.0</distortionK1>
+        <distortionK2>0.0</distortionK2>
+        <distortionK3>0.0</distortionK3>
+        <distortionT1>0.0</distortionT1>
+        <distortionT2>0.0</distortionT2>
+      </plugin>
+    </sensor>
+  </gazebo>
 </robot>

Commit message: new fingertips w/ mods for stable grasp; requires more iters in gazebo launch file

File: dvrk_model/model/gazebo_psm.tool.sca.urdf.xacro (robot description, xacro)
@@ -85,12 +85,10 @@
         </geometry>
       </visual>
-      <collision>
+      <!--collision>
         <origin rpy="0 0 0" xyz="0 0 0"/>
           <geometry>
-              <!-- coarse model; a simple box -->
-              <!--box size="0.05 0.2 0.05"/-->
           <mesh filename="package://dvrk_model/meshes/psm/tool_wrist_sca_link_2.dae"/>
           </geometry>
-      </collision>
+      </collision-->
      <selfCollide>true</selfCollide>
     <inertial>
@@ -120,22 +118,112 @@
         </geometry>
       </visual>
-      <collision>
+      <!--collision>
         <origin rpy="0 3.1516 0" xyz="0 0 0"/>
           <geometry>
-              <!-- coarse model; a simple box -->
-              <!--box size="0.05 0.2 0.05"/-->
           <mesh filename="package://dvrk_model/meshes/psm/tool_wrist_sca_link_2.dae"/>
           </geometry>
+      </collision-->
+     <selfCollide>false</selfCollide>
+    <inertial>
+      <origin xyz="0 0 0" rpy="0 0 0"/>
+      <mass value="0.05"/>
+      <inertia
+        ixx="0.01" ixy="0.0" ixz="0.0"
+        iyy="0.01" iyz="0.0"
+        izz="0.005"/>
+    </inertial>
+    </link>
+<!-- wsn: try adding a fingertip for grasping -->
+    <link name="${prefix}fingertip2">
+     <visual>
+        <origin rpy="0 0 0" xyz="0.001 0.005 0.0005"/>
+        <geometry>
+          <box size="0.002 0.01 0.004"/>
+        </geometry>
+     </visual>
+      <collision>
+        <origin rpy="0 0 0" xyz="0.001 0.005 0.0005"/>
+        <geometry>
+          <box size="0.002 0.01 0.004"/>
+        </geometry>
+       <surface>
+            <friction>
+              <ode>
+                <mu>30.0</mu>
+                <mu2>30.0</mu2>
+              </ode>
+            </friction>
+            <contact>
+              <ode>
+                <kp>1000000.0</kp>
+                <kd>100.0</kd>
+                <max_vel>1.0</max_vel>
+                <min_depth>0.001</min_depth>
+              </ode>
+            </contact>
+          </surface>
       </collision>
-     <selfCollide>true</selfCollide>
-    <inertial>
-      <origin xyz="0 0 0" rpy="0 0 0"/>
-      <mass value="0.05"/>
-      <inertia
-        ixx="0.01" ixy="0.0" ixz="0.0"
-        iyy="0.01" iyz="0.0"
-        izz="0.005"/>
-    </inertial>
-    </link>
+     <inertial>
+      <origin xyz="0 0 0" rpy="0 0 0"/>
+      <mass value="0.05"/>
+      <inertia
+        ixx="0.01" ixy="0.0" ixz="0.0"
+        iyy="0.01" iyz="0.0"
+        izz="0.005"/>
+    </inertial>
+    </link>
+    <!-- attach fingertip pad  -->
+    <joint name="${prefix}fingertip2_joint" type="fixed">
+      <parent link="${prefix}tool_wrist_sca_ee_link_2"/>
+      <child link="${prefix}fingertip2"/>
+      <axis xyz="0 0 1"/>
+      <origin rpy="0 0 0" xyz="0 0 0"/>
+    </joint>
+<!-- wsn: other fingertip -->
+    <link name="${prefix}fingertip1">
+     <visual>
+        <origin rpy="0 0 0" xyz="-0.001 0.005 0.0005"/>
+        <geometry>
+          <box size="0.002 0.01 0.004"/>
+        </geometry>
+     </visual>
+      <collision>
+        <origin rpy="0 0 0" xyz="-0.001 0.005 0.0005"/>
+        <geometry>
+          <box size="0.002 0.01 0.004"/>
+        </geometry>
+       <surface>
+            <friction>
+              <ode>
+                <mu>30.0</mu>
+                <mu2>30.0</mu2>
+              </ode>
+            </friction>
+            <contact>
+              <ode>
+                <kp>1000000.0</kp>
+                <kd>100.0</kd>
+                <max_vel>1.0</max_vel>
+                <min_depth>0.001</min_depth>
+              </ode>
+            </contact>
+          </surface>
+      </collision>
+     <inertial>
+      <origin xyz="0 0 0" rpy="0 0 0"/>
+      <mass value="0.05"/>
+      <inertia
+        ixx="0.01" ixy="0.0" ixz="0.0"
+        iyy="0.01" iyz="0.0"
+        izz="0.005"/>
+    </inertial>
+    </link>
+    <!-- attach fingertip pad 1  -->
+    <joint name="${prefix}fingertip1_joint" type="fixed">
+      <parent link="${prefix}tool_wrist_sca_ee_link_1"/>
+      <child link="${prefix}fingertip1"/>
+      <axis xyz="0 0 1"/>
+      <origin rpy="0 0 0" xyz="0 0 0"/>
+    </joint>
     <!-- tool tip -->
     <joint name="${prefix}tool_tip_joint_" type="fixed">

Commit message: tweaking davinci gazebo model; should merge in manipulation branch

File: dvrk_model/model/gazebo_psm.tool.sca.urdf.xacro (robot description, xacro)
@@ -80,16 +80,28 @@
     <link name="${prefix}tool_wrist_sca_ee_link_1">
       <visual>
-        <origin rpy="0 0 0" xyz="0 0 0"/>
-        <geometry>
-          <mesh filename="package://dvrk_model/meshes/psm/tool_wrist_sca_link_2.dae"/>
-        </geometry>
-      </visual>
-      <collision>
+        <!--origin rpy="0 0 0" xyz="0 0 0"/-->
+        <origin rpy="-1.5708 0 0" xyz="0 0 0"/>
+        <geometry>
+          <!--mesh filename="package://dvrk_model/meshes/psm/tool_wrist_sca_link_2.dae"/-->
+          <mesh filename="package://dvrk_model/meshes/psm/finger.dae"/>
+        </geometry>
+      </visual>
+      <collision>
+        <!--origin rpy="0 0 0" xyz="0 0 0"/-->
         <origin rpy="0 0 0" xyz="0 0 0"/>
           <geometry>
               <!-- coarse model; a simple box -->
               <!--box size="0.05 0.2 0.05"/-->
-          <mesh filename="package://dvrk_model/meshes/psm/tool_wrist_sca_link_2.dae"/>
-          </geometry>
+          <!--mesh filename="package://dvrk_model/meshes/psm/tool_wrist_sca_link_2.dae"/-->
+          <mesh filename="package://dvrk_model/meshes/psm/finger.dae"/>
+          </geometry>
+          <surface>
+            <friction>
+            <ode>
+              <mu>0.2</mu>
+              <mu2>0.2</mu2>
+            </ode>
+            </friction>
+          </surface>
       </collision>
      <selfCollide>true</selfCollide>
@@ -103,4 +115,45 @@
     </inertial>
     </link>
+ <!-- wsn: try adding some fingertip pads, to experiment with friction, etc -->
+    <link name="${prefix}fingertip1">
+      <visual>
+        <!--origin rpy="0 0 0" xyz="0 0 0"/-->
+        <origin rpy="0 0 0" xyz="0 0.005 0"/>
+        <geometry>
+          <box size="0.0001 0.01 0.003"/>
+        </geometry>
+      </visual>
+      <collision>
+        <!--origin rpy="0 0 0" xyz="0 0 0"/-->
+        <origin rpy="0 0 0" xyz="0 0 0"/>
+          <geometry>
+                       <box size="0.001 0.02 0.003"/>
+          </geometry>
+          <gazebo>
+          <surface>
+            <friction>
+            <ode>
+              <mu>0.2</mu>
+              <mu2>0.2</mu2>
+            </ode>
+            </friction>
+          </surface>
+          </gazebo>
+      </collision>
+     <inertial>
+      <origin xyz="0 0 0" rpy="0 0 0"/>
+      <mass value="0.005"/>
+      <inertia
+        ixx="0.01" ixy="0.0" ixz="0.0"
+        iyy="0.01" iyz="0.0"
+        izz="0.005"/>
+     </inertial>
+    </link>
+    <joint name="${prefix}fingertip_connector1" type="fixed">
+      <parent link="${prefix}tool_wrist_sca_ee_link_1"/>
+      <child link="${prefix}fingertip1"/>
+      <axis xyz="0 0 1"/>
+      <origin rpy="0 0 0" xyz="0 0 0"/>
+    </joint>
     <!-- joint 7-2: Outer open angle 2   -->
     <joint name="${prefix}outer_wrist_open_angle_joint_mimic" type="revolute">
@@ -115,16 +168,26 @@
     <link name="${prefix}tool_wrist_sca_ee_link_2">
       <visual>
-        <origin rpy="0 3.1516 0" xyz="0 0 0"/>
-        <geometry>
-          <mesh filename="package://dvrk_model/meshes/psm/tool_wrist_sca_link_2.dae"/>
-        </geometry>
-      </visual>
-      <collision>
-        <origin rpy="0 3.1516 0" xyz="0 0 0"/>
-          <geometry>
-              <!-- coarse model; a simple box -->
-              <!--box size="0.05 0.2 0.05"/-->
-          <mesh filename="package://dvrk_model/meshes/psm/tool_wrist_sca_link_2.dae"/>
-          </geometry>
+        <!--origin rpy="0 3.1516 0" xyz="0 0 0"/-->
+                <origin rpy="-1.5708 3.1516 0" xyz="0 0 0"/>
+        <geometry>
+          <!--mesh filename="package://dvrk_model/meshes/psm/tool_wrist_sca_link_2.dae"/-->
+          <mesh filename="package://dvrk_model/meshes/psm/finger.dae"/>
+        </geometry>
+      </visual>
+      <collision>
+        <!--origin rpy="0 3.1516 0" xyz="0 0 0"/-->
+        <origin rpy="-1.5708 3.1516 0" xyz="0 0 0"/>
+          <geometry>
+          <!--mesh filename="package://dvrk_model/meshes/psm/tool_wrist_sca_link_2.dae"/-->
+           <mesh filename="package://dvrk_model/meshes/psm/finger.dae"/>
+          </geometry>
+      <surface>
+        <friction>
+          <ode>
+            <mu>0.2</mu>
+            <mu2>0.2</mu2>
+          </ode>
+        </friction>
+      </surface>
       </collision>
      <selfCollide>true</selfCollide>
@@ -155,5 +218,17 @@
   <gazebo reference="${prefix}tool_tip_link">
     <material>Gazebo/Red</material>
+    <!-- try adding some friction to enable fingers to grip objects -->
   </gazebo>
+  <!--
+    <gazebo reference="${prefix}tool_wrist_sca_ee_link_2">
+    <mu1>0.2</mu1>
+    <mu2>0.2</mu2>
+  </gazebo>
+    </gazebo>
+    <gazebo reference="${prefix}tool_wrist_sca_ee_link_1">
+    <mu1>0.2</mu1>
+    <mu2>0.2</mu2>
+  </gazebo>
+-->
  <transmission name="${prefix}tran5">
     <type>transmission_interface/SimpleTransmission</type>

Commit message: progress towards simulated stereo. W/ camera syncer, managed to get stereo calib results in .yaml files.  Seem reasonable.
can turn 1mm peg blue to distinguish it in color images.
need to put models in .gazebo

File: dvrk_model/model/gazebo_psm.tool.sca.urdf.xacro (robot description, xacro)
@@ -85,13 +85,4 @@
         </geometry>
       </visual>
-      <!--collision>
-        <origin rpy="0 0 0" xyz="0 0 0"/>
-          <geometry>
-              <!-- coarse model; a simple box -->
-              <!--box size="0.05 0.2 0.05"/-->
-          <mesh filename="package://dvrk_model/meshes/psm/tool_wrist_sca_link_2.dae"/>
-          </geometry>
-      </collision-->
-     <selfCollide>true</selfCollide>
     <inertial>
       <origin xyz="0 0 0" rpy="0 0 0"/>
