Commit message: fixes to collision model; created gazebo launch for davinci w/ table and pin; made new cartesian playfile pgm that interprets gripper poses w/rt left camera optical frame.

File: dvrk_model/model/gazebo_psm.base.urdf.xacro (robot description, xacro)
@@ -234,12 +234,4 @@
         </geometry>
       </visual>
-      <collision>
-        <origin rpy="0 0 1.5708" xyz="0 0 0.041"/>
-          <geometry>
-              <!-- coarse model; a simple box -->
-              <!--box size="0.05 0.2 0.05"/-->
-          <mesh filename="package://dvrk_model/meshes/psm/tool_main.dae"/>
-          </geometry>
-      </collision>
       <inertial>
       <origin xyz="0 0 0" rpy="0 0 0"/>
@@ -268,12 +260,4 @@
         </geometry>
       </visual>
-      <collision>
-        <origin rpy="0 0 1.5708" xyz="0 0 0.041"/>
-          <geometry>
-              <!-- coarse model; a simple box -->
-              <!--box size="0.05 0.2 0.05"/-->
-          <mesh filename="package://dvrk_model/meshes/psm/tool_wrist_link.dae"/>
-          </geometry>
-      </collision>
     <inertial>
       <origin xyz="0 0 0" rpy="0 0 0"/>
@@ -299,12 +283,4 @@
           <mesh filename="package://dvrk_model/meshes/psm/tool_wrist_shaft_link.dae"/>
         </geometry>
-      <collision>
-        <origin rpy="0 0 1.5708" xyz="0 0 0.041"/>
-          <geometry>
-              <!-- coarse model; a simple box -->
-              <!--box size="0.05 0.2 0.05"/-->
-          <mesh filename="package://dvrk_model/meshes/psm/tool_wrist_shaft_link.dae"/>
-          </geometry>
-      </collision>
       </visual>
     <inertial>

File: dvrk_model/model/gazebo_psm.tool.sca.urdf.xacro (robot description, xacro)
@@ -33,5 +33,5 @@
           </geometry>
       </collision>
-     <selfCollide>true</selfCollide>
+     <selfCollide>false</selfCollide>
     <inertial>
       <origin xyz="0 0 0" rpy="0 0 0"/>
@@ -85,13 +85,4 @@
         </geometry>
       </visual>
-      <!--collision>
-        <origin rpy="0 0 0" xyz="0 0 0"/>
-          <geometry>
-              <!-- coarse model; a simple box -->
-              <!--box size="0.05 0.2 0.05"/-->
-          <mesh filename="package://dvrk_model/meshes/psm/tool_wrist_sca_link_2.dae"/>
-          </geometry>
-      </collision-->
-     <selfCollide>true</selfCollide>
     <inertial>
       <origin xyz="0 0 0" rpy="0 0 0"/>
@@ -120,11 +111,4 @@
         </geometry>
       </visual>
-      <!--collision>
-        <origin rpy="0 3.1516 0" xyz="0 0 0"/>
-          <geometry>
-          <mesh filename="package://dvrk_model/meshes/psm/tool_wrist_sca_link_2.dae"/>
-          </geometry>
-      </collision-->
-     <selfCollide>false</selfCollide>
     <inertial>
       <origin xyz="0 0 0" rpy="0 0 0"/>

File: dvrk_model/model/wsn_both_psms.urdf.xacro (robot description, xacro)
@@ -9,5 +9,5 @@
       <parent link="world"/>
       <child link="camera"/>
-      <origin rpy="0.0 0.0 0.0" xyz="0.0 0.0 0.5"/>
+      <origin rpy="0.0 0.0 0.0" xyz="0.0 0.0 0.4"/>
   </joint>
     <link name="camera">
@@ -139,5 +139,6 @@
         <imageTopicName>image_raw</imageTopicName>
         <cameraInfoTopicName>camera_info</cameraInfoTopicName>
-        <frameName>left_camera_link</frameName>
+        <frameName>left_camera_optical_frame</frameName>
+        <!--frameName>left_camera_link</frameName-->
         <hackBaseline>0.07</hackBaseline>
         <distortionK1>0.0</distortionK1>
